File: H0BR40/Design/H0BR40.brd (EAGLE design)
At the start: 34.6 x 30 mm, 30 parts, among them P1 HEXABIT_17.32, U1 STM32F091CBU6, U2 LSM6DS3TR-C, U3 LSM303AGRTR, X1 XTALL_CSTCE8M00G52

Commit message: in this commit: - renamed all res and caps to match circuitmaker original design - fixed BOM files (note: in circuit maker and website C15 should be C14) - regenerated documentation and all output files
Parts:
- C1: value 10nF -> 100nF
- C3: value 100nF -> 4.7uF; device Hexabitz:C-0603 -> Hexabitz:C-0805-POL
- C5: value 100nF -> 10nF
- C7: value 4.7uF -> 100nF; device Hexabitz:C-0805-POL -> Hexabitz:C-0603
- R2: value 0.0R -> 10.0K
- R3: value 10.0K -> 0.0R
- moved C8 16.5 mm to (28.8, 29.7), turned to 0 degrees
- moved C6 13.6 mm to (37.4, 40.4), turned to 90 degrees
- moved C5 13.1 mm to (40.7, 31.8)
- moved C3 12.1 mm to (27.9, 32.9), turned to 270 degrees
- moved R2 12.0 mm to (35.2, 40.3), turned to 270 degrees
- moved R3 12.0 mm to (45.9, 34.9), turned to 0 degrees
- moved C4 6.98 mm to (27.4, 39.8), turned to 90 degrees
- moved C1 6.50 mm to (43.2, 37.8)
- moved C7 2.51 mm to (29.5, 38.6)
Connections:
- net B1: now also R2.2; no longer R3.2
- net GND: now also C1.2; no longer C5.2
- net R1: now also C1.1; no longer C8.1
- net VDD: now also C8.1; no longer C5.1
- net VDDA: now also C5.1; no longer C1.1
- net VSSA: now also C5.2, R3.2; no longer C1.2, R2.2
