File: H0BR40/Design/H0BR40.sch (EAGLE design)
At the start: 30 parts, among them P1 HEXABIT_17.32, U1 STM32F091CBU6, U2 LSM6DS3TR-C, U3 LSM303AGRTR, X1 XTALL_CSTCE8M00G52

Commit message: in this commit: - renamed all res and caps to match circuitmaker original design - fixed BOM files (note: in circuit maker and website C15 should be C14) - regenerated documentation and all output files
Parts:
- C1: value 10nF -> 100nF; CAPACITANCE 10nF -> 100nF; MFN KEMET -> AVX; MPN C0603C103K5RACTU -> 0603YC104K4T2A; OCTOPART_URL https://octopart.com/c0603c103k5ractu-kemet-133094?r=sp&s=R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 -> https://octopart.com/0603yc104k4t2a-avx+interconnect+%2F+el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; VOLTAGE_RATING 50V -> 16.0 V
- C2: MFN Yageo -> AVX; MPN CC0805KKX7R7BB105 -> TAJR105M016RNJ; OCTOPART_URL https://octopart.com/cc0805kkx7r7bb105-yageo-8376555?r=sp&s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 -> http://octopart.com/tajr105m016rnj-avx-1188552; VOLTAGE_RATING 16V -> 16.0 V
- C3: value 100nF -> 4.7uF; device Hexabitz:C-0603 -> Hexabitz:C-0805-POL; CAPACITANCE 100nF -> 4.7uF; MFN KEMET -> Panasonic; MPN C0603C104K8RACTU -> 10TPU4R7MSI; OCTOPART_URL https://octopart.com/c0603c104k8ractu-kemet-145075?r=sp&s=9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 -> https://octopart.com/10tpu4r7msi-panasonic-29487748; TOLERANCE 10% -> 20%; VOLTAGE_RATING 10V -> 10.0 V
- C4: MFN Murata -> Panasonic; MPN GRM21BC81E475KA12L -> 10TPU4R7MSI; OCTOPART_URL https://octopart.com/grm21bc81e475ka12l-murata-10331911?r=s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 -> https://octopart.com/10tpu4r7msi-panasonic-29487748; VOLTAGE_RATING 25V -> 10 V
- C5: value 100nF -> 10nF; CAPACITANCE 100nF -> 10nF; MFN KEMET -> AVX; MPN C0603C104K8RACTU -> 0603YC103KAT4A; OCTOPART_URL https://octopart.com/c0603c104k8ractu-kemet-145075?r=sp&s=9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 -> https://octopart.com/0603yc103kat4a-avx+interconnect+%2F+el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; VOLTAGE_RATING 10 -> 16.0 V
- C6, C8: MFN KEMET -> AVX; MPN C0603C104K8RACTU -> 0603YC104K4T2A; OCTOPART_URL https://octopart.com/c0603c104k8ractu-kemet-145075?r=sp&s=9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 -> https://octopart.com/0603yc104k4t2a-avx+interconnect+%2F+el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; VOLTAGE_RATING 10V -> 16.0 V
- C7: value 4.7uF -> 100nF; device Hexabitz:C-0805-POL -> Hexabitz:C-0603; CAPACITANCE 4.7uF -> 100nF; MFN Murata -> AVX; MPN GRM21BC81E475KA12L -> 0603YC104K4T2A; OCTOPART_URL https://octopart.com/grm21bc81e475ka12l-murata-10331911?r=s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 -> https://octopart.com/0603yc104k4t2a-avx+interconnect+%2F+el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; VOLTAGE_RATING 25V -> 16.0 V
- C9: MFN KEMET -> AVX; MPN C0603C104K8RACTU -> 0603YC104K4T2A; OCTOPART_URL https://octopart.com/c0603c104k8ractu-kemet-145075?r=sp&s=9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 -> https://octopart.com/0603yc104k4t2a-avx+interconnect+%2F+el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; TOLERANCE 10V -> 16.0 V
- R1: MFN Yageo -> Panasonic; MPN RC0603FR-07270RL -> ERJ-3GEYJ271V; OCTOPART_URL https://octopart.com/search?q=RC0603FR-07270RL&start=0 -> https://octopart.com/erj-3geyj271v-panasonic-55560546; TOLERANCE 1% -> 5%
- R2: value 0.0R -> 10.0K; MFN Yageo -> Vishay; MPN RC0603JR-070RL -> CRCW060310K0JNEB; OCTOPART_URL https://octopart.com/rc0603jr-070rl-yageo-1241539?r=sp&s=X2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 -> https://octopart.com/crcw060310k0jneb-vishay-46603269; RESISTANCE 0.0 Ohm -> 10.0K Ohm; TOLERANCE (none) -> 5%
- R3: value 10.0K -> 0.0R; MFN Yageo -> Vishay; MPN RC0603JR-0710KL -> CRCW06030000Z0EAHP; OCTOPART_URL https://octopart.com/search?q=RC0603JR-0710KL&start=0 -> https://octopart.com/crcw06030000z0eahp-vishay-44320230; RESISTANCE 10.0K Ohm -> 0.0 Ohm; TOLERANCE 5% -> (none)
Connections:
- net B1: now also R2.2; no longer R3.2
- net GND: now also C1.2, C3.-, C7.2; no longer C3.2, C5.2, C7.-
- net R1: now also C1.1; no longer C8.1
- net VDD: now also C3.+, C7.1, C8.1; no longer C3.1, C5.1, C7.+
- net VDDA: now also C5.1; no longer C1.1
- net VSSA: now also C5.2, R3.2; no longer C1.2, R2.2
Other:
- moved on the sheet: C1, C4, C5, C6, C8, R2, R3
